File: mavhi/mavhi-hardware/mavhi-hardware/mavhi-hardware.kicad_sch (KiCad schematic)
At the start: 5 parts, among them M1 Stepper_Motor_unipolar_5pin, SW1 SW_Push, SW2 SW_Push, U1 ULN2003

Commit message: feat: update poster, applause, hardware and part2
Parts:
- added D1, D2, D3, D4: LED, symbol Device:LED
- added R1, R2, R3, R4: 100, symbol Device:R
- added U2: 74HC595, symbol 74xx:74HC595
Connections:
- net +5V: now also U2.10 (~{SRCLR}), U2.16 (VCC)
- net GND: now also D1.1 (K), D2.1 (K), D3.1 (K), D4.1 (K), U2.13 (~{OE}), U2.8 (GND)
- net Shift_01_Data: now reaches A1.19 (D4)
- net Shift_01_Data: now also U2.14 (SER)
- net Shift_01_Clock: now reaches A1.20 (D5)
- net Shift_01_Clock: now also U2.11 (SRCLK)
- net Shift_01_Latch: now reaches A1.21 (D6)
- net Shift_01_Latch: now also U2.12 (RCLK)
- net A0: no longer names the net of A1.9 (A0)
- net A1: no longer names the net of A1.10 (A1)
- net A2: no longer names the net of A1.11 (A2)
- new net: D2.2 (A), R2.1
- new net: R2.2, U2.2 (QC)
- new net: D1.2 (A), R1.1
- new net: R1.2, U2.3 (QD)
- new net: D3.2 (A), R3.1
- new net: D4.2 (A), R4.1
- new net: R4.2, U2.15 (QA)
- new net: R3.2, U2.1 (QB)
